File: DP02.kicad_sch (KiCad schematic)
At the start: 15 parts

Commit message: Starting DP03
Parts:
- removed E11, E20, E24, E38, E60: MC10101, symbol DEC20:MC10101
- removed E13, E15, E25, E32: MC10141, symbol DEC20:MC10141
- removed E35, E45, E48: MC10174, symbol DEC20:MC10174
- removed E49, E55, E56: MC10164, symbol DEC20:MC10164
Other:
- title: DATA PATH ARX & MQ REGISTERS -> (none)

Commit message: Added DP02
Parts:
- added E11, E20, E24, E38, E60: MC10101, symbol DEC20:MC10101
- added E13, E15, E25, E32: MC10141, symbol DEC20:MC10141
- added E35, E45, E48: MC10174, symbol DEC20:MC10174
- added E49, E55, E56: MC10164, symbol DEC20:MC10164
Connections:
- new net: E35.7 (SEL1), E38.6 (Bout), E45.7 (SEL1), E48.7 (SEL1)
- new net: E49.10 (SEL4), E55.10 (SEL4), E56.10 (SEL4), E60.5 (Aout)
- new net: E49.7 (SEL1), E55.7 (SEL1), E56.7 (SEL1), E60.9 (Dout)
- new net: E49.9 (SEL2), E55.9 (SEL2), E56.9 (SEL2), E60.6 (Bout)
- new net: E13.10 (S1), E15.10 (S1), E20.6 (Bout)
- new net: E24.14 (~Cout), E25.10 (S1), E25.7 (S2)
- new net: E35.9 (SEL2), E38.5 (Aout), E45.9 (SEL2), E48.9 (SEL2)
- new net: E15.5 (SHFT-3IN), E20.11 (Cout)
- new net: E13.7 (S2), E15.7 (S2), E20.5 (Aout)
- new net: E35.14 (EN), E38.15 (~Dout), E45.14 (EN), E48.14 (EN)
- new net: E35.10 (D13), E35.6 (D03), E38.9 (Dout), E45.10 (D13), E45.6 (D03), E48.10 (D13), E48.6 (D03)
- new net: E13.5 (SHFT-3IN), E20.9 (Dout)
- new net: E32.10 (S1), E32.7 (S2)
- new net AA1: E11.13 (Din), E24.13 (Din), E25.3 (Q3), E32.3 (Q3)
- new net AC1: E11.7 (Bin), E24.7 (Bin), E25.2 (Q2), E32.2 (Q2)
- new net AD 0 H: E45.4 (D02), E49.14 (D7), E55.4 (D2)
- new net AD 1 H: E45.12 (D12), E56.4 (D2)
- new net AD 2 H: E48.4 (D02), E49.4 (D2), E56.12 (D5)
- new net AD 3 H: E48.12 (D12), E49.12 (D5)
- new net AD 4 H: E35.4 (D02)
- new net AD 5 H: E35.12 (D12)
- new net ADX 0 H: E55.13 (D6)
- new net ADX 1 H: E55.12 (D5), E56.13 (D6)
- new net ADX 2 H: E49.13 (D6)
- new net AJ2: E11.4 (Ain), E24.4 (Ain), E25.14 (Q0), E25.15 (Q1), E32.14 (Q0), E32.15 (Q1)
- new net ARM 0 H: E55.15 (B)
- new net ARM 1 H: E56.15 (B)
- new net ARM 2 H: E49.15 (B)
- new net ARMM 1 H: E56.6 (D0)
- new net ARMM 2 H: E49.6 (D0)
- new net ARX 0 A H: E24.5 (Aout)
- new net ARX 1 A H: E24.6 (Bout)
- new net ARX 2 A H: E24.9 (Dout)
- new net ARX 3 A H: E11.5 (Aout)
- new net ARX 4 A H: E11.6 (Bout)
- new net ARX 5 A H: E11.9 (Dout)
- new net ARXM 0 H: E25.11 (D1), E25.12 (D0)
- new net ARXM 1 H: E25.9 (D2), E32.12 (D0)
- new net ARXM 2 H: E25.6 (D3)
- new net ARXM 3 H: E32.11 (D1)
- new net ARXM 4 H: E32.9 (D2)
- new net ARXM 5 H: E32.6 (D3)
- new net BR1: E24.10 (Cin)
- new net BU2: E20.7 (Bin)
- new net BV2: E20.4 (Ain)
- new net CA1: E35.11 (D11)
- new net CACHE DATA 0 B H: E55.5 (D1)
- new net CACHE DATA 1 B H: E56.5 (D1)
- new net CACHE DATA 2 B H: E49.5 (D1)
- new net CD1: E20.10 (Cin)
- new net CD2: E13.14 (Q0), E48.3 (D00), E55.3 (D3)
- new net CS1: E15.2 (Q2), E20.13 (Din)
- new net DA1: E48.11 (D11)
- new net DE2: E35.5 (D01)
- new net DF1: E15.3 (Q3)
- new net DF2: E45.13 (D10)
- new net DK2: E55.14 (D7)
- new net DP04 CLK C H: E13.4 (CLK)
- new net DP04 CLK D H: E15.4 (CLK)
- new net DP04 CLK E H: E25.4 (CLK)
- new net DP04 CLK F H: E32.4 (CLK)
- new net DS1: E48.5 (D01), E49.11 (D4)
- new net DS2: E56.3 (D3)
- new net DT2: E49.3 (D3)
- new net EC1: E45.11 (D11), E56.11 (D4)
- new net ED1: E45.5 (D01), E55.11 (D4)
- new net EL2: E56.14 (D7)
- new net FD2: E60.7 (Bin)
- new net FF1: E45.3 (D00), E60.4 (Ain)
- new net FJ1: E60.13 (Din)
- new net MQ 1 H: E13.15 (Q1), E48.13 (D10)
- new net MQ 2 H: E13.2 (Q2), E35.3 (D00)
- new net MQ 3 H: E15.15 (Q1), E35.13 (D10)
- new net MQM 0 H: E13.12 (D0), E45.2 (B0)
- new net MQM 1 H: E13.11 (D1), E13.13 (SHFT-0IN), E45.15 (B1)
- new net MQM 2 H: E13.9 (D2), E15.12 (D0), E48.2 (B0)
- new net MQM 3 H: E13.6 (D3), E15.11 (D1), E15.13 (SHFT-0IN), E48.15 (B1)
- new net MQM 4 H: E15.9 (D2), E35.2 (B0)
- new net MQM 5 H: E15.6 (D3), E35.15 (B1)
- new net VCC1: E11.1 (VCC1), E11.1 (VCC1), E11.1 (VCC1), E20.1 (VCC1), E20.1 (VCC1), E20.1 (VCC1), E20.1 (VCC1), E24.1 (VCC1), E24.1 (VCC1), E24.1 (VCC1), E24.1 (VCC1), E35.1 (VCC1), E38.1 (VCC1), E38.1 (VCC1), E38.1 (VCC1), E45.1 (VCC1), E48.1 (VCC1), E60.1 (VCC1), E60.1 (VCC1), E60.1 (VCC1)
- new net VCC2: E11.16 (VCC2), E11.16 (VCC2), E11.16 (VCC2), E20.16 (VCC2), E20.16 (VCC2), E20.16 (VCC2), E20.16 (VCC2), E24.16 (VCC2), E24.16 (VCC2), E24.16 (VCC2), E24.16 (VCC2), E35.16 (VCC2), E38.16 (VCC2), E38.16 (VCC2), E38.16 (VCC2), E45.16 (VCC2), E48.16 (VCC2), E60.16 (VCC2), E60.16 (VCC2), E60.16 (VCC2)
- new net VEE: E35.8 (VEE), E45.8 (VEE), E48.8 (VEE)
Other:
- title: (none) -> DATA PATH ARX & MQ REGISTERS
