File: DP02.kicad_sch (KiCad schematic)
At the start: 18 parts

Commit message: Convert all backplane refs to global labels and stick them on J1 pins. Convert all signal labels to global labels too so they are "global" inside M8512 board.
Connections:
- net AS1 renamed ARX 1 A H
- net AS2 renamed ARX 0 A H
- net CC1 renamed CACHE DATA 5 B H
- net CJ2 renamed ADX 0 H
- net CM2 renamed ARX 1 B H
- net CP1 renamed AD 4 H
- net DD1 renamed CACHE DATA 3 B H
- net DK1 renamed ADX 4 H
- net DL1 renamed AD 1 H
- net DL2 renamed CACHE DATA 4 B H
- net DN1 renamed CTL MQM EN H
- net DR1 renamed AD 3 H
- net DR2 renamed AD 2 H
- net ED2 renamed CACHE DATA 1 B H
- net EE2 renamed CACHE DATA 2 B H
- net EL1 renamed AD 5 H
- net EM1 renamed CACHE DATA 0 B H
- net EP2 renamed AD 0 H
- net ES1 renamed ADX 5 H

Commit message: Testing some verilog for KiCadVerilog
Parts:
- E60: VerilogCode (none) -> MC10101(COMin, nAout, Aout, Ain, nBout, Bout, Bin, nCout, C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; VerilogInclude (none) -> MC10101.v
Changed lines of the file:
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@@
+      (effects (font (size 1.27 1.27)) hide)
+    )
+    (property "VerilogInclude" "MC10101.v" (id 4) (at 50.165 118.11 0)
+      (effects (font (size 1.27 1.27)) hide)
+    )
+    (property "VerilogCode" "MC10101(COMin, nAout, Aout, Ain, nBout, Bout, Bin, nCout, Cout, Cin, nDout, Dout, Din);" (id 5) (at 50.165 118.11 0)
       (effects (font (size 1.27 1.27)) hide)
     )

Commit message: checkpoint
Parts:
- E60: VerilogCode MC10101(COMin, nAout, Aout, Ain, nBout, Bout, Bin, nCout, C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 -> (none); VerilogInclude MC10101.v -> (none)
Changed lines of the file:
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@@
-      (effects (font (size 1.27 1.27)) hide)
-    )
-    (property "VerilogInclude" "MC10101.v" (id 4) (at 50.165 118.11 0)
-      (effects (font (size 1.27 1.27)) hide)
-    )
-    (property "VerilogCode" "MC10101(COMin, nAout, Aout, Ain, nBout, Bout, Bin, nCout, Cout, Cin, nDout, Dout, Din);" (id 5) (at 50.165 118.11 0)
       (effects (font (size 1.27 1.27)) hide)
     )

Commit message: checkpoint
Connections:
- net AA1 renamed ARX 5 H <AA1>
- net ARX 5 H <AA1>: no longer E24.13 (Din)
- net AC1 renamed ARX 4 H <AC1>
- net ARX 4 H <AC1>: no longer E24.7 (Bin)
- net AD 0 H renamed AD 0 H <EP2>
- net AD 1 H renamed AD 1 H <DL1>
- net AD 2 H renamed AD 2 H <DR2>
- net AD 3 H renamed AD 3 H <DR1>
- net AD 4 H renamed AD 4 H <CP1>
- net AD 5 H renamed AD 5 H <EL1>
- net ADX 0 H renamed ADX 0 H <CJ2>
- net ADX 4 H renamed ADX 4 H <DK1>
- net ADX 5 H renamed ADX 5 H <ES1>
- net AJ2 renamed ARX 3 H <AJ2>
- net ARX 3 H <AJ2>: no longer E24.4 (Ain)
- net ARX 0 A H renamed ARX 0 A H <AS2>
- net ARX 1 A H renamed ARX 1 A H <AS1>
- net ARX 1 B H renamed ARX 1 B H <CM2>
- net BR1 renamed CTL ARX LOAD H <BR1>
- net BU2 renamed CTL MQ SEL 1 H <BU2>
- net CTL MQ SEL 1 H <BU2>: no longer E38.7 (Bin)
- net BV2 renamed CTL MQ SEL 2 H <BV2>
- net CTL MQ SEL 2 H <BV2>: no longer E38.4 (Ain)
- net CA1 renamed SH 5 H <CA1>
- net CACHE DATA 0 B H renamed CACHE DATA 0 B H <EM1>
- net CACHE DATA 1 B H renamed CACHE DATA 1 B H <ED2>
- net CACHE DATA 2 B H renamed CACHE DATA 2 B H <EE2>
- net CACHE DATA 3 B H renamed CACHE DATA 3 B H <DD1>
- net CACHE DATA 4 B H renamed CACHE DATA 4 B H <DL2>
- net CACHE DATA 5 B H renamed CACHE DATA 5 B H <CC1>
- net CD1 renamed <CD1>
- net CD2 renamed MQ 0 H <CD2>
- net CJ1 renamed <CJ1>
- net CS1 renamed MQ 4 H <CS1>
- net CS2 renamed <CS2>
- net CTL MQM EN H renamed CTL MQM EN H <DN1>
- net DA1 renamed SH 3 H <DA1>
- net DE2 renamed SH 4 H <DE2>
- net DF1 renamed MQ 5 H <DF1>
- net DF2 renamed <DF2>
- net DK2 renamed <DK2>
- net DS1 renamed SH 2 H <DS1>
- net EC1 renamed SH 1 H <EC1>
- net ED1 renamed SH 0 H <ED1>
- net ES2 renamed <ES2>
- net FD2 renamed <FD2>
- net FF1 renamed <FF1>
- net FJ1 renamed <FJ1>
- new net ARX 0 H <AJ2>: E24.4 (Ain)
- new net ARX 1 H <AC1>: E24.7 (Bin)
- new net ARX 2 H <AA1>: E24.13 (Din)
- new net CTL MQ SEL 1 H <DJ1>: E38.7 (Bin)
- new net CTL MQ SEL 2 H <DM1>: E38.4 (Ain)
