File: DP02.kicad_sch (KiCad schematic)
At the start: 18 parts

Commit message: Nearly done switching to <ABn> backplane labels
Connections:
- net ARX 1 B H <CM2>: no longer E25.14 (Q0)
- net ARX 3 H <AJ2>: no longer E25.15 (Q1)
- net ARX 4 H <AC1>: no longer E25.2 (Q2)
- net ARX 5 H <AA1>: no longer E25.3 (Q3)
- net ARX 0 H <AJ2> renamed ARX 0 H <EJ2>
- net ARX 0 H <EJ2>: now also E25.15 (Q1)
- net ARX 1 H <AC1> renamed ARX 1 H <BD2>
- net ARX 1 H <BD2>: now also E25.2 (Q2)
- net ARX 2 H <AA1> renamed ARX 2 H <DC1>
- net ARX 2 H <DC1>: now also E25.3 (Q3)
- new net ARX 1 B H <BR2>: E25.14 (Q0)
Changed lines of the file:
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@@
     )
   )
-  (global_label "ARX 1 B H <CM2>" (shape input) (at 225.425 48.26 0) (fields_autoplaced)
-    (effects (font (size 1.27 1.27)) (justify left))
-    (property "Intersheet References" "${INTERSHEET_REFS}" (id 0) (at 246.1624 48.1806 0)
+  (global_label "ARX 1 B H <BR2>" (shape input) (at 225.425 48.26 0) (fields_autoplaced)
+    (effects (font (size 1.27 1.27)) (justify left))
+    (property "Intersheet References" "${INTERSHEET_REFS}" (id 0) (at 245.981 48.1806 0)
       (effects (font (size 1.27 1.27)) (justify left) hide)
     )
@@
     )
   )
-  (global_label "ARX 4 H <AC1>" (shape input) (at 225.425 55.88 0) (fields_autoplaced)
-    (effects (font (size 1.27 1.27)) (justify left))
-    (property "Intersheet References" "${INTERSHEET_REFS}" (id 0) (at 243.5619 55.8006 0)
+  (global_label "ARX 1 H <BD2>" (shape input) (at 225.425 55.88 0) (fields_autoplaced)
+    (effects (font (size 1.27 1.27)) (justify left))
+    (property "Intersheet References" "${INTERSHEET_REFS}" (id 0) (at 243.7433 55.8006 0)
       (effects (font (size 1.27 1.27)) (justify left) hide)
     )
@@
     )
   )
-  (global_label "ARX 0 H <AJ2>" (shape input) (at 267.335 43.815 180) (fields_autoplaced)
-    (effects (font (size 1.27 1.27)) (justify right))
-    (property "Intersheet References" "${INTERSHEET_REFS}" (id 0) (at 249.5005 43.7356 0)
+  (global_label "ARX 0 H <EJ2>" (shape input) (at 267.335 43.815 180) (fields_autoplaced)
+    (effects (font (size 1.27 1.27)) (justify right))
+    (property "Intersheet References" "${INTERSHEET_REFS}" (id 0) (at 249.44 43.7356 0)
       (effects (font (size 1.27 1.27)) (justify right) hide)
     )
@@
     )
   )
-  (global_label "ARX 3 H <AJ2>" (shape input) (at 225.425 52.07 0) (fields_autoplaced)
-    (effects (font (size 1.27 1.27)) (justify left))
-    (property "Intersheet References" "${INTERSHEET_REFS}" (id 0) (at 243.2595 51.9906 0)
+  (global_label "ARX 0 H <EJ2>" (shape input) (at 225.425 52.07 0) (fields_autoplaced)
+    (effects (font (size 1.27 1.27)) (justify left))
+    (property "Intersheet References" "${INTERSHEET_REFS}" (id 0) (at 243.32 51.9906 0)
       (effects (font (size 1.27 1.27)) (justify left) hide)
     )
@@
     )
   )
-  (global_label "ARX 5 H <AA1>" (shape input) (at 225.425 59.69 0) (fields_autoplaced)
-    (effects (font (size 1.27 1.27)) (justify left))
-    (property "Intersheet References" "${INTERSHEET_REFS}" (id 0) (at 243.3805 59.6106 0)
-      (effects (font (size 1.27 1.27)) (justify left) hide)
-    )
-  )
-  (global_label "ARX 2 H <AA1>" (shape input) (at 267.335 61.595 180) (fields_autoplaced)
-    (effects (font (size 1.27 1.27)) (justify right))
-    (property "Intersheet References" "${INTERSHEET_REFS}" (id 0) (at 249.3795 61.5156 0)
+  (global_label "ARX 2 H <DC1>" (shape input) (at 225.425 59.69 0) (fields_autoplaced)
+    (effects (font (size 1.27 1.27)) (justify left))
+    (property "Intersheet References" "${INTERSHEET_REFS}" (id 0) (at 243.7433 59.6106 0)
+      (effects (font (size 1.27 1.27)) (justify left) hide)
+    )
+  )
+  (global_label "ARX 2 H <DC1>" (shape input) (at 267.335 61.595 180) (fields_autoplaced)
+    (effects (font (size 1.27 1.27)) (justify right))
+    (property "Intersheet References" "${INTERSHEET_REFS}" (id 0) (at 249.0167 61.5156 0)
       (effects (font (size 1.27 1.27)) (justify right) hide)
     )
@@
     )
   )
-  (global_label "ARX 1 H <AC1>" (shape input) (at 267.335 52.705 180) (fields_autoplaced)
-    (effects (font (size 1.27 1.27)) (justify right))
-    (property "Intersheet References" "${INTERSHEET_REFS}" (id 0) (at 249.1981 52.6256 0)
-      (effects (font (size 1.27 1.27)) (justify right) hide)
-    )
+  (global_label "ARX 1 H <BD2>" (shape input) (at 267.335 52.705 180) (fields_autoplaced)
+    (effects (font (size 1.27 1.27)) (justify right))
+    (property "Intersheet References" "${INTERSHEET_REFS}" (id 0) (at 249.0167 52.6256 0)
+      (effects (font (size 1.27 1.27)) (justify right) hide)
+    )

Commit message: Fix a bunch of typos and their backplane signal names
Connections:
- net ARX 1 B H <BR2> renamed ARX 0 B H <BR2>
- net CTL MQ SEL 1 H <DJ1> renamed CTL MQM SEL 1 H <DJ1>
- net CTL MQ SEL 2 H <DM1> renamed CTL MQM SEL 2 H <DM1>
Changed lines of the file:
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@@
     )
   )
-  (global_label "ARX 1 B H <BR2>" (shape input) (at 225.425 48.26 0) (fields_autoplaced)
+  (global_label "ARX 0 B H <BR2>" (shape input) (at 225.425 48.26 0) (fields_autoplaced)
     (effects (font (size 1.27 1.27)) (justify left))
     (property "Intersheet References" "${INTERSHEET_REFS}" (id 0) (at 245.981 48.1806 0)
@@
     )
   )
-  (global_label "CTL MQ SEL 2 H <DM1>" (shape input) (at 112.395 181.61 180) (fields_autoplaced)
-    (effects (font (size 1.27 1.27)) (justify right))
-    (property "Intersheet References" "${INTERSHEET_REFS}" (id 0) (at 86.0938 181.5306 0)
+  (global_label "CTL MQM SEL 2 H <DM1>" (shape input) (at 112.395 181.61 180) (fields_autoplaced)
+    (effects (font (size 1.27 1.27)) (justify right))
+    (property "Intersheet References" "${INTERSHEET_REFS}" (id 0) (at 84.6424 181.5306 0)
       (effects (font (size 1.27 1.27)) (justify right) hide)
     )
@@
     )
   )
-  (global_label "CTL MQ SEL 1 H <DJ1>" (shape input) (at 112.395 190.5 180) (fields_autoplaced)
-    (effects (font (size 1.27 1.27)) (justify right))
-    (property "Intersheet References" "${INTERSHEET_REFS}" (id 0) (at 86.5776 190.4206 0)
-      (effects (font (size 1.27 1.27)) (justify right) hide)
-    )
+  (global_label "CTL MQM SEL 1 H <DJ1>" (shape input) (at 112.395 190.5 180) (fields_autoplaced)
+    (effects (font (size 1.27 1.27)) (justify right))
+    (property "Intersheet References" "${INTERSHEET_REFS}" (id 0) (at 85.1262 190.4206 0)
+      (effects (font (size 1.27 1.27)) (justify right) hide)
+    )

Commit message: Fix a bunch of typos, add ${N} macros for slot specific net names
Connections:
- net ARXM 2 H is gone; now on net ARXM ${N+2} H: E49.15 (B)
- net AD 0 H <EP2> renamed AD ${N+0} H <EP2>
- net AD 1 H <DL1> renamed AD ${N+1} H <DL1>
- net AD 2 H <DR2> renamed AD ${N+2} H <DR2>
- net AD 3 H <DR1> renamed AD ${N+3} H <DR1>
- net AD 4 H <CP1> renamed AD ${N+4} H <CP1>
- net AD 5 H <EL1> renamed AD ${N+5} H <EL1>
- net ADX 0 H <CJ2> renamed ADX ${N+0} H <CJ2>
- net ADX 1 H renamed ADX ${N+1} H
- net ADX 2 H renamed ADX ${N+2} H
- net ADX 3 H renamed ADX ${N+3} H
- net ADX 4 H <DK1> renamed ADX ${N+4} H <DK1>
- net ADX 5 H <ES1> renamed ADX ${N+5} H <ES1>
- net ARMX 2 H renamed ARXM ${N+2} H
- net ARX 0 A H <AS2> renamed ARX ${N+0} A H <AS2>
- net ARX 0 B H <BR2> renamed ARX ${N+0} B H <BR2>
- net ARX 0 H <EJ2> renamed ARX ${N+0} H <EJ2>
- net ARX 1 A H <AS1> renamed ARX ${N+1} A H <AS1>
- net ARX 1 B H <CM2> renamed ARX ${N+1} B H <CM2>
- net ARX 1 H <BD2> renamed ARX ${N+1} H <BD2>
- net ARX 2 A H renamed ARX ${N+2} A H
- net ARX 2 H <DC1> renamed ARX ${N+2} H <DC1>
- net ARX 3 A H renamed ARX ${N+3} A H
- net ARX 3 H <AJ2> renamed ARX ${N+3} H <AJ2>
- net ARX 4 A H renamed ARX ${N+4} A H
- net ARX 4 H <AC1> renamed ARX ${N+4} H <AC1>
- net ARX 5 A H renamed ARX ${N+5} A H
- net ARX 5 H <AA1> renamed ARX ${N+5} H <AA1>
- net ARXM 0 H renamed ARXM ${N+0} H
- net ARXM 1 H renamed ARXM ${N+1} H
- net ARXM 3 H renamed ARXM ${N+3} H
- net ARXM 4 H renamed ARXM ${N+4} H
- net ARXM 5 H renamed ARXM ${N+5} H
- net CACHE DATA 0 B H <EM1> renamed CACHE DATA ${N+0} B H <EM1>
- net CACHE DATA 1 B H <ED2> renamed CACHE DATA ${N+1} B H <ED2>
- net CACHE DATA 2 B H <EE2> renamed CACHE DATA ${N+2} B H <EE2>
- net CACHE DATA 3 B H <DD1> renamed CACHE DATA ${N+3} B H <DD1>
- net CACHE DATA 4 B H <DL2> renamed CACHE DATA ${N+4} B H <DL2>
- net CACHE DATA 5 B H <CC1> renamed CACHE DATA ${N+5} B H <CC1>
- net MQ 0 H <CD2> renamed MQ ${N+0} H <CD2>
- net MQ 1 H renamed MQ ${N+1} H
- net MQ 2 H renamed MQ ${N+2} H
- net MQ 3 H renamed MQ ${N+3} H
- net MQ 4 H <CS1> renamed MQ ${N+4} H <CS1>
- net MQ 5 H <DF1> renamed MQ ${N+5} H <DF1>
- net MQM 0 H renamed MQM ${N+0} H
- net MQM 1 H renamed MQM ${N+1} H
- net MQM 2 H renamed MQM ${N+2} H
- net MQM 3 H renamed MQM ${N+3} H
- net MQM 4 H renamed MQM ${N+4} H
- net MQM 5 H renamed MQM ${N+5} H
- net SH 0 H <ED1> renamed SH ${N+0} H <ED1>
- net SH 1 H <EC1> renamed SH ${N+1} H <EC1>
- net SH 2 H <DS1> renamed SH ${N+2} H <DS1>
- net SH 3 H <DA1> renamed SH ${N+3} H <DA1>
- net SH 4 H <DE2> renamed SH ${N+4} H <DE2>
- net SH 5 H <CA1> renamed SH ${N+5} H <CA1>
Other:
- moved on the sheet: E11A, E11B, E11D, E13, E15, E20A, E20B, E20C, E20D, E24A, E24B, E24C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

Commit message: Now DP02 is done, but still need to do DP03/4 and relabel J1 net names to match.
Connections:
- net <CD1> renamed ${N/30+1, MQ ${N+6} h, AD CRY -02 A H} <CD1>
- net <CJ1> renamed ${N/30+1, ADX ${N+6} H, MQ 00 H} <CJ1>
- net <CS2> renamed ${(N+199)/100, ADX 34 H, MQ ${N-2} H} <CS2>
- net <DF2> renamed ${(N+199)/100, ADX 35 H, MQ ${N-1} H} <DF2>
- net <DK2> renamed ${(N+199)/100, AD 34 H, ADX ${N-2} H} <DK2>
- net <ES2> renamed ${(N+199)/100, AD 35 H, AX ${N-1} H} <ES2>
- net <FD2> renamed ${N/18+1, CTL ARXML SEL 2 H, CTL ARXR SEL 2 H} <FD2>
- net <FF1> renamed ${CRAM ARXML SEL 4 ${N/18+1,00,06} H <FF1>
- net <FJ1> renamed ${N/18+1, CTL ARXL SEL 1 H, CTL ARXR SEL 1 H} <FJ1>
Other:
- moved on the sheet: E55

Commit message: Get rid of errors between J1 net name and pages
Connections:
- net ${CRAM ARXML SEL 4 ${N/18+1,00,06} H <FF1> renamed CRAM ARXML SEL 4 ${N/18+1,00,06} H <FF1>
Changed lines of the file:
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@@
     )
   )
-  (global_label "${CRAM ARXML SEL 4 ${N{slash}18+1,00,06} H <FF1>" (shape input) (at 30.48 81.915 0) (fields_autoplaced)
+  (global_label "CRAM ARXML SEL 4 ${N{slash}18+1,00,06} H <FF1>" (shape input) (at 30.48 81.915 0) (fields_autoplaced)
     (effects (font (size 1.27 1.27)) (justify left))
-    (property "Intersheet References" "${INTERSHEET_REFS}" (id 0) (at 86.5355 81.8356 0)
+    (property "Intersheet References" "${INTERSHEET_REFS}" (id 0) (at 84.4793 81.8356 0)
       (effects (font (size 1.27 1.27)) (justify left) hide)
     )

Commit message: Remove "slash" in several places as an experiment. it did not work.
Connections:
- net ${(N+199)/100, AD 34 H, ADX ${N-2} H} <DK2> renamed ${(N+199)/100, AD 34 H, ADX ${N-2} H} <DK2>
- net ${(N+199)/100, AD 35 H, AX ${N-1} H} <ES2> renamed ${(N+199)/100, AD 35 H, AX ${N-1} H} <ES2>
- net ${(N+199)/100, ADX 34 H, MQ ${N-2} H} <CS2> renamed ${(N+199)/100, ADX 34 H, MQ ${N-2} H} <CS2>
- net ${(N+199)/100, ADX 35 H, MQ ${N-1} H} <DF2> renamed ${(N+199)/100, ADX 35 H, MQ ${N-1} H} <DF2>
- net ${N/18+1, CTL ARXL SEL 1 H, CTL ARXR SEL 1 H} <FJ1> renamed ${N/18+1, CTL ARXL SEL 1 H, CTL ARXR SEL 1 H} <FJ1>
- net ${N/18+1, CTL ARXML SEL 2 H, CTL ARXR SEL 2 H} <FD2> renamed ${N/18+1, CTL ARXML SEL 2 H, CTL ARXR SEL 2 H} <FD2>
- net ${N/30+1, ADX ${N+6} H, MQ 00 H} <CJ1> renamed ${N/30+1, ADX ${N+6} H, MQ 00 H} <CJ1>
- net ${N/30+1, MQ ${N+6} h, AD CRY -02 A H} <CD1> renamed ${N/30+1, MQ ${N+6} h, AD CRY -02 A H} <CD1>
- net CRAM ARXML SEL 4 ${N/18+1,00,06} H <FF1> renamed CRAM ARXML SEL 4 ${N/18+1,00,06} H <FF1>
Changed lines of the file:
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@@
     )
   )
-  (global_label "${N{slash}18+1, CTL ARXML SEL 2 H, CTL ARXR SEL 2 H} <FD2>" (shape input)
+  (global_label "${N/18+1, CTL ARXML SEL 2 H, CTL ARXR SEL 2 H} <FD2>" (shape input)
     (at 30.48 77.47 0) (fields_autoplaced)
     (effects (font (size 1.27 1.27)) (justify left))
@@
     )
   )
-  (global_label "${N{slash}18+1, CTL ARXL SEL 1 H, CTL ARXR SEL 1 H} <FJ1>" (shape input)
+  (global_label "${N/18+1, CTL ARXL SEL 1 H, CTL ARXR SEL 1 H} <FJ1>" (shape input)
     (at 30.48 73.025 0) (fields_autoplaced)
     (effects (font (size 1.27 1.27)) (justify left))
@@
     )
   )
-  (global_label "${(N+199){slash}100, ADX 34 H, MQ ${N-2} H} <CS2>" (shape input) (at 102.235 150.495 180) (fields_autoplaced)
+  (global_label "${(N+199)/100, ADX 34 H, MQ ${N-2} H} <CS2>" (shape input) (at 102.235 150.495 180) (fields_autoplaced)
     (effects (font (size 1.27 1.27)) (justify right))
     (property "Intersheet References" "${INTERSHEET_REFS}" (id 0) (at 45.0909 150.4156 0)
@@
     )
   )
-  (global_label "${N{slash}30+1, ADX ${N+6} H, MQ 00 H} <CJ1>" (shape input) (at 375.92 132.715 180) (fields_autoplaced)
+  (global_label "${N/30+1, ADX ${N+6} H, MQ 00 H} <CJ1>" (shape input) (at 375.92 132.715 180) (fields_autoplaced)
     (effects (font (size 1.27 1.27)) (justify right))
     (property "Intersheet References" "${INTERSHEET_REFS}" (id 0) (at 324.3398 132.6356 0)
@@
     )
   )
-  (global_label "${(N+199){slash}100, AD 35 H, AX ${N-1} H} <ES2>" (shape input) (at 135.255 133.985 180) (fields_autoplaced)
+  (global_label "${(N+199)/100, AD 35 H, AX ${N-1} H} <ES2>" (shape input) (at 135.255 133.985 180) (fields_autoplaced)
     (effects (font (size 1.27 1.27)) (justify right))
     (property "Intersheet References" "${INTERSHEET_REFS}" (id 0) (at 79.9252 133.9056 0)
@@
     )
   )
-  (global_label "CRAM ARXML SEL 4 ${N{slash}18+1,00,06} H <FF1>" (shape input) (at 30.48 81.915 0) (fields_autoplaced)
+  (global_label "CRAM ARXML SEL 4 ${N/18+1,00,06} H <FF1>" (shape input) (at 30.48 81.915 0) (fields_autoplaced)
     (effects (font (size 1.27 1.27)) (justify left))
     (property "Intersheet References" "${INTERSHEET_REFS}" (id 0) (at 84.4793 81.8356 0)
@@
     )
   )
-  (global_label "${N{slash}30+1, MQ ${N+6} h, AD CRY -02 A H} <CD1>" (shape input)
-    (at 343.535 217.805 0) (fields_autoplaced)
+  (global_label "${N/30+1, MQ ${N+6} h, AD CRY -02 A H} <CD1>" (shape input) (at 343.535 217.805 180) (fields_autoplaced)
     (effects (font (size 1.27 1.27)) (justify right))
     (property "Intersheet References" "${INTERSHEET_REFS}" (id 0) (at 284.8186 217.7256 0)
@@
     )
   )
-  (global_label "${(N+199){slash}100, AD 34 H, ADX ${N-2} H} <DK2>" (shape input) (at 81.28 87.63 180) (fields_autoplaced)
+  (global_label "${(N+199)/100, AD 34 H, ADX ${N-2} H} <DK2>" (shape input) (at 81.28 87.63 180) (fields_autoplaced)
     (effects (font (size 1.27 1.27)) (justify right))
     (property "Intersheet References" "${INTERSHEET_REFS}" (id 0) (at 24.4988 87.5506 0)
@@
     )
   )
-  (global_label "${(N+199){slash}100, ADX 35 H, MQ ${N-1} H} <DF2>" (shape input) (at 102.235 161.925 180) (fields_autoplaced)
+  (global_label "${(N+199)/100, ADX 35 H, MQ ${N-1} H} <DF2>" (shape input) (at 102.235 161.925 180) (fields_autoplaced)
     (effects (font (size 1.27 1.27)) (justify right))
     (property "Intersheet References" "${INTERSHEET_REFS}" (id 0) (at 45.2119 161.8456 0)
