File: M8513-YA-CSH.kicad_sch (KiCad schematic)
At the start: 0 parts

Commit message: EDP is "done" but there is still much work to do to standardize and set up netlist export and verilog creation
Other:
- title: (none) -> DATA PATH AR REGISTER
Changed lines of the file:
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@@
 (kicad_sch (version 20211123) (generator eeschema)
-  (paper "A4")
+  (paper "B")
   (title_block
+    (title "DATA PATH AR REGISTER")
     (date "10/21/1976")
+    (rev "A")
     (company "DIGITAL")
+    (comment 1 "M8512-0-DP01")
   )
 )
