File: DP04.kicad_sch (KiCad schematic)
At the start: 26 parts

Commit message: I think all pages now have ${N+x} stuff, but still need to relabel J1 net names to match.
Connections:
- net <CE2> renamed ${N/18+1, CON FM WRITE 00-17 L, CON FM WRITE 18-35 L} <CE2>
- net <FE2> renamed ${N/18+1, CTL AD TO EBUS L H, CTL AD TO EBUS R} <FE2>
- net AR ${N+0}A H <FJ2> renamed AR ${N+0} A H <FJ2>
Changed lines of the file:
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@@
     (stroke (width 0) (type default) (color 0 0 0 0))
   )
-  (wire (pts (xy 144.145 41.91) (xy 145.415 41.91))
+  (wire (pts (xy 142.875 38.1) (xy 145.415 41.91))
     (stroke (width 0) (type default) (color 0 0 0 0))
   )
@@
     (stroke (width 0) (type default) (color 0 0 0 0))
   )
-  (wire (pts (xy 375.92 41.91) (xy 376.555 41.91))
+  (wire (pts (xy 374.65 37.465) (xy 376.555 41.91))
     (stroke (width 0) (type default) (color 0 0 0 0))
   )
@@
     (stroke (width 0) (type default) (color 0 0 0 0))
   )
-  (wire (pts (xy 260.35 41.91) (xy 260.985 41.91))
+  (wire (pts (xy 258.445 37.465) (xy 260.985 41.91))
     (stroke (width 0) (type default) (color 0 0 0 0))
   )
@@
     (stroke (width 0) (type default) (color 0 0 0 0))
   )
+  (wire (pts (xy 86.995 100.965) (xy 50.8 100.965))
+    (stroke (width 0) (type default) (color 0 0 0 0))
+  )
   (wire (pts (xy 356.235 107.315) (xy 360.045 107.315))
     (stroke (width 0) (type default) (color 0 0 0 0))
@@
     (stroke (width 0) (type default) (color 0 0 0 0))
   )
+  (wire (pts (xy 86.995 107.315) (xy 86.995 100.965))
+    (stroke (width 0) (type default) (color 0 0 0 0))
+  )
   (wire (pts (xy 122.555 163.83) (xy 122.555 161.29))
     (stroke (width 0) (type default) (color 0 0 0 0))
@@
     (stroke (width 0) (type default) (color 0 0 0 0))
   )
-  (wire (pts (xy 318.135 41.91) (xy 318.77 41.91))
+  (wire (pts (xy 316.865 38.1) (xy 318.77 41.91))
     (stroke (width 0) (type default) (color 0 0 0 0))
   )
@@
     (stroke (width 0) (type default) (color 0 0 0 0))
   )
+  (wire (pts (xy 50.8 100.965) (xy 50.8 96.52))
+    (stroke (width 0) (type default) (color 0 0 0 0))
+  )
   (wire (pts (xy 203.2 64.77) (xy 260.985 64.77))
     (stroke (width 0) (type default) (color 0 0 0 0))
@@
     (stroke (width 0) (type default) (color 0 0 0 0))
   )
-  (wire (pts (xy 201.93 41.91) (xy 203.2 41.91))
+  (wire (pts (xy 200.66 38.1) (xy 203.2 41.91))
     (stroke (width 0) (type default) (color 0 0 0 0))
   )
@@
   )
   (wire (pts (xy 201.295 133.35) (xy 228.6 133.35))
+    (stroke (width 0) (type default) (color 0 0 0 0))
+  )
+  (wire (pts (xy 85.725 107.315) (xy 86.995 107.315))
     (stroke (width 0) (type default) (color 0 0 0 0))
   )
@@
     )
   )
-  (global_label "AR ${N+5} H" (shape input) (at 375.92 41.91 180) (fields_autoplaced)
-    (effects (font (size 1.27 1.27)) (justify right))
-    (property "Intersheet References" "${INTERSHEET_REFS}" (id 0) (at 366.6731 41.8306 0)
+  (global_label "AR ${N+5} H" (shape input) (at 374.65 37.465 180) (fields_autoplaced)
+    (effects (font (size 1.27 1.27)) (justify right))
+    (property "Intersheet References" "${INTERSHEET_REFS}" (id 0) (at 365.4031 37.3856 0)
       (effects (font (size 1.27 1.27)) (justify right) hide)
     )
@@
     )
   )
-  (global_label "<FE2>" (shape input) (at 50.8 96.52 180) (fields_autoplaced)
-    (effects (font (size 1.27 1.27)) (justify right))
-    (property "Intersheet References" "${INTERSHEET_REFS}" (id 0) (at 41.795 96.4406 0)
+  (global_label "${N{slash}18+1, CTL AD TO EBUS L H, CTL AD TO EBUS R} <FE2>" (shape input)
+    (at 85.725 107.315 0) (fields_autoplaced)
+    (effects (font (size 1.27 1.27)) (justify right))
+    (property "Intersheet References" "${INTERSHEET_REFS}" (id 0) (at 18.3605 107.2356 0)
       (effects (font (size 1.27 1.27)) (justify right) hide)
     )
@@
     )
   )
-  (global_label "AR ${N+2} H" (shape input) (at 201.93 41.91 180) (fields_autoplaced)
-    (effects (font (size 1.27 1.27)) (justify right))
-    (property "Intersheet References" "${INTERSHEET_REFS}" (id 0) (at 192.6831 41.8306 0)
+  (global_label "AR ${N+2} H" (shape input) (at 200.66 38.1 180) (fields_autoplaced)
+    (effects (font (size 1.27 1.27)) (justify right))
+    (property "Intersheet References" "${INTERSHEET_REFS}" (id 0) (at 191.4131 38.0206 0)
       (effects (font (size 1.27 1.27)) (justify right) hide)
     )
@@
     )
   )
-  (global_label "AR ${N+4} H" (shape input) (at 318.135 41.91 180) (fields_autoplaced)
-    (effects (font (size 1.27 1.27)) (justify right))
-    (property "Intersheet References" "${INTERSHEET_REFS}" (id 0) (at 308.8881 41.8306 0)
+  (global_label "AR ${N+4} H" (shape input) (at 316.865 38.1 180) (fields_autoplaced)
+    (effects (font (size 1.27 1.27)) (justify right))
+    (property "Intersheet References" "${INTERSHEET_REFS}" (id 0) (at 307.6181 38.0206 0)
       (effects (font (size 1.27 1.27)) (justify right) hide)
     )
@@
     )
   )
-  (global_label "AR ${N+1} H <BL2>" (shape input) (at 144.145 41.91 180) (fields_autoplaced)
-    (effects (font (size 1.27 1.27)) (justify right))
-    (property "Intersheet References" "${INTERSHEET_REFS}" (id 0) (at 127.2781 41.8306 0)
-      (effects (font (size 1.27 1.27)) (justify right) hide)
-    )
-  )
-  (global_label "<CE2>" (shape input) (at 121.92 167.64 180) (fields_autoplaced)
-    (effects (font (size 1.27 1.27)) (justify right))
-    (property "Intersheet References" "${INTERSHEET_REFS}" (id 0) (at 112.7336 167.5606 0)
+  (global_label "AR ${N+1} H <BL2>" (shape input) (at 142.875 38.1 180) (fields_autoplaced)
+    (effects (font (size 1.27 1.27)) (justify right))
+    (property "Intersheet References" "${INTERSHEET_REFS}" (id 0) (at 126.0081 38.0206 0)
+      (effects (font (size 1.27 1.27)) (justify right) hide)
+    )
+  )
+  (global_label "${N{slash}18+1, CON FM WRITE 00-17 L, CON FM WRITE 18-35 L} <CE2>" (shape input)
+    (at 121.92 167.64 0) (fields_autoplaced)
+    (effects (font (size 1.27 1.27)) (justify right))
+    (property "Intersheet References" "${INTERSHEET_REFS}" (id 0) (at 46.0283 167.5606 0)
       (effects (font (size 1.27 1.27)) (justify right) hide)
     )
@@
     )
   )
-  (global_label "AR ${N+3} H" (shape input) (at 260.35 41.91 180) (fields_autoplaced)
-    (effects (font (size 1.27 1.27)) (justify right))
-    (property "Intersheet References" "${INTERSHEET_REFS}" (id 0) (at 251.1031 41.8306 0)
+  (global_label "AR ${N+3} H" (shape input) (at 258.445 37.465 180) (fields_autoplaced)
+    (effects (font (size 1.27 1.27)) (justify right))
+    (property "Intersheet References" "${INTERSHEET_REFS}" (id 0) (at 249.1981 37.3856 0)
       (effects (font (size 1.27 1.27)) (justify right) hide)
     )
@@
     )
   )
-  (global_label "AR ${N+0}A H <FJ2>" (shape input) (at 99.695 203.2 180) (fields_autoplaced)
-    (effects (font (size 1.27 1.27)) (justify right))
-    (property "Intersheet References" "${INTERSHEET_REFS}" (id 0) (at 79.8043 203.1206 0)
-      (effects (font (size 1.27 1.27)) (justify right) hide)
-    )
+  (global_label "AR ${N+0} A H <FJ2>" (shape input) (at 99.695 203.2 180) (fields_autoplaced)
+    (effects (font (size 1.27 1.27)) (justify right))
+    (property "Intersheet References" "${INTERSHEET_REFS}" (id 0) (at 75.2081 203.1206 0)
+      (effects (font (size 1.27 1.27)) (justify right) hide)
+    )

Commit message: Remove "slash" in several places as an experiment. it did not work.
Connections:
- net ${N/18+1, CON FM WRITE 00-17 L, CON FM WRITE 18-35 L} <CE2> renamed ${N/18+1, CON FM WRITE 00-17 L, CON FM WRITE 18-35 L} <CE2>
- net ${N/18+1, CTL AD TO EBUS L H, CTL AD TO EBUS R} <FE2> renamed ${N/18+1, CTL AD TO EBUS L H, CTL AD TO EBUS R} <FE2>
Changed lines of the file:
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@@
     )
   )
-  (global_label "${N{slash}18+1, CTL AD TO EBUS L H, CTL AD TO EBUS R} <FE2>" (shape input)
+  (global_label "${N/18+1, CTL AD TO EBUS L H, CTL AD TO EBUS R} <FE2>" (shape input)
     (at 85.725 107.315 0) (fields_autoplaced)
     (effects (font (size 1.27 1.27)) (justify right))
@@
     )
   )
-  (global_label "${N{slash}18+1, CON FM WRITE 00-17 L, CON FM WRITE 18-35 L} <CE2>" (shape input)
+  (global_label "${N/18+1, CON FM WRITE 00-17 L, CON FM WRITE 18-35 L} <CE2>" (shape input)
     (at 121.92 167.64 0) (fields_autoplaced)
     (effects (font (size 1.27 1.27)) (justify right))

Commit message: Parser is greedily eating characters up to next "}" instead of following nesting. Fix lowercase "h" found in some signal names. Add error message stuff for signal name syntax errors.
Connections:
- net ${N/18+1, CON FM WRITE 00-17 L, CON FM WRITE 18-35 L} <CE2> renamed ${N/18+1,CON FM WRITE 00-17 L,CON FM WRITE 18-35 L} <CE2>
- net ${N/18+1, CTL AD TO EBUS L H, CTL AD TO EBUS R} <FE2> renamed ${N/18+1,CTL AD TO EBUS L H,CTL AD TO EBUS R} <FE2>
Changed lines of the file:
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@@
     )
   )
-  (global_label "${N/18+1, CTL AD TO EBUS L H, CTL AD TO EBUS R} <FE2>" (shape input)
+  (global_label "${N/18+1,CTL AD TO EBUS L H,CTL AD TO EBUS R} <FE2>" (shape input)
     (at 85.725 107.315 0) (fields_autoplaced)
     (effects (font (size 1.27 1.27)) (justify right))
@@
     )
   )
-  (global_label "${N/18+1, CON FM WRITE 00-17 L, CON FM WRITE 18-35 L} <CE2>" (shape input)
+  (global_label "${N/18+1,CON FM WRITE 00-17 L,CON FM WRITE 18-35 L} <CE2>" (shape input)
     (at 121.92 167.64 0) (fields_autoplaced)
     (effects (font (size 1.27 1.27)) (justify right))
